File: hard/powerpic.kicad_sch (KiCad schematic)
At the start: 21 parts, among them U1 PIC16LF1919x-I/MR

Commit message: Version 1.1 Release
Parts:
- removed TP10: RH0, ppc-watch:TestPoint_Pad_D0.5mm, symbol Connector:TestPoint
- PPC1: footprint ppc-watch:ppc-board -> powerpic:ppc-board; symbol ppc-watch:ppc-board -> powerpic:ppc-board
- TP1, TP2, TP3, TP4, TP5: footprint ppc-watch:Progo_Pad_D2.0mm -> powerpic:Progo_Pad_D2.0mm; now left out of the parts list
- TP6: value RG7 -> GND; footprint ppc-watch:TestPoint_Pad_D0.5mm -> powerpic:Progo_Pad_D2.0mm; now left out of the parts list
- TP7: value RA3 -> ADJ; footprint ppc-watch:TestPoint_Pad_D0.5mm -> powerpic:Progo_Pad_D2.0mm; now left out of the parts list
- TP8: value RA2 -> MODE; footprint ppc-watch:TestPoint_Pad_D0.5mm -> powerpic:Progo_Pad_D2.0mm; now left out of the parts list
- TP9: value RH1 -> BUZZ; footprint ppc-watch:TestPoint_Pad_D0.5mm -> powerpic:Progo_Pad_D2.0mm; now left out of the parts list
- U1: symbol ppc-watch:PIC16F1919x-xMR -> powerpic:PIC16F1919x-xMR
Connections:
- net ADJ: now also TP7.1
- net BUZZ: now also TP9.1, U1.19 (COM7/SEG15/RG7); no longer U1.18 (SEG41/RF0)
- net GND: now also TP6.1
- net MODE: now also TP8.1
- net RH1: no longer TP9.1
- net ROW0: now also U1.24 (RA0/SEG33); no longer U1.28 (RA4/SEG14)
- net ROW1: now also U1.23 (RA1/SEG18); no longer U1.27 (RA5)
- net ROW2: now also U1.22 (RA2/SEG34); no longer U1.24 (RA0/SEG33)
- net ROW3: now also U1.21 (RA3/SEG35); no longer U1.23 (RA1/SEG18)
- removed net RA2: TP8.1, U1.22 (RA2/SEG34)
- removed net RA3: TP7.1, U1.21 (RA3/SEG35)
- removed net RG7: TP6.1, U1.19 (COM7/SEG15/RG7)
Other:
- note added: "(6x) 2mm Dia Spaced 2.5mm"
- note added: "BUZ"
- note added: "GND"
- note removed: "(5x) 0.5mm Dia"
- note removed: "(5x) 2mm Dia Spaced 2.5mm"
- note removed: "Unused Pins"
- moved on the sheet: TP1, TP2, TP3, TP4, TP5
