File: hardware/powerpic.kicad_pcb (KiCad board)
At the start: 2 copper layers, 25.6 x 27.6 mm, 17 parts, among them U1 PIC16LF1919x-I/MR, Y1 32.768kHz

Commit message: Starting work on version 3 of the hardware.
Routing:
- net VCC: track 35.0 -> 0.00 mm, vias 2 -> 0
- net Net-(D1-A): track 32.7 -> 0.00 mm, vias 2 -> 0
- net /SEG12: track 22.4 -> 0.00 mm, vias 2 -> 0
- net /SEG13: track 22.0 -> 0.00 mm, vias 2 -> 0
- net /SEG14: track 19.6 -> 0.00 mm, vias 2 -> 0
- net /MODE: track 19.5 -> 0.00 mm, vias 1 -> 0
- net /~{MCLR}: track 19.1 -> 0.00 mm, vias 1 -> 0
- net /SOSCO: track 18.9 -> 0.00 mm, vias 2 -> 0
- net /COM0: track 18.8 -> 0.00 mm, vias 2 -> 0
- net /SEG11: track 18.0 -> 0.00 mm, vias 2 -> 0
- net /SOSCI: track 17.8 -> 0.00 mm, vias 2 -> 0
- net /COM1: track 17.5 -> 0.00 mm, vias 2 -> 0
- net /SEG9: track 17.1 -> 0.00 mm, vias 2 -> 0
- net /COM2: track 16.6 -> 0.00 mm, vias 2 -> 0
- net /SEG10: track 16.5 -> 0.00 mm, vias 2 -> 0
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- removed copper zone on B.Cu, net GND
- removed copper zone on F.Cu, net GND
Other:
- board text added: "TODO"
- board text removed: "2.0"
- board text removed: "BUZ"
- board text removed: "C"
- board text removed: "D"
- board text removed: "DBG"
- board text removed: "Designed by Rex McKinnon in Oakland CA"
- board text removed: "GND"
- board text removed: "ICSP"
- board text removed: "Manufactured by JLCPCB in May 2022"
- board text removed: "PowerPIC"
- board text removed: "R"
- board text removed: "VIN"
