File: hardware/powerpic.kicad_pcb (KiCad board)
At the start: 2 copper layers, 25.6 x 27.6 mm, 19 parts, among them U1 PIC16LF1919x-I/MR, Y1 32.768kHz

Commit message: Release hardware version 3.0
Parts:
- added D2: D_Filled, Diode_SMD:D_SOD-882, F.Cu at (139.8, 63.4)
- added R2: 600, Resistor_SMD:R_0402_1005Metric, F.Cu at (139.7, 65.7)
- moved kibuzzard-6619F682 0.50 mm to (133.9, 50.2)
Connections:
- net /DEBUG renamed /CASE
Routing:
- net VCC: track 35.0 -> 40.4 mm, vias 2 -> 3
- net Net-(D2-K): track 0.00 -> 2.33 mm
- net /VLCD3: track 8.77 -> 7.06 mm
- net /SEG12: track 22.4 -> 21.3 mm
- net /CASE: track 2.90 -> 4.04 mm
- net /SEG11: track 18.0 -> 16.9 mm
- net /SEG9: track 17.1 -> 16.2 mm
- net /SEG10: track 16.5 -> 15.7 mm
- net GND: vias 38 -> 52
- added copper zone on In1.Cu, net GND
- added copper zone on In2.Cu, net GND
Other:
- copper layers 2 -> 4
- board text added: "2631"
- board text added: "3.0"
- board text added: "ML2016 BATTERY ONLY"
- board text added: "[!]"
- board text added: "v3.0"
- board text removed: "2416"
- board text removed: "v2.1"
