File: hardware/powerpic.kicad_sch (KiCad schematic)
At the start: 13 parts, among them U1 PIC16LF1919x-I/MR, Y1 32.768kHz

Commit message: Release hardware version 3.0
Parts:
- added D2: D_Filled, Diode_SMD:D_SOD-882, symbol Device:D_Filled
- added R2: 680, Resistor_SMD:R_0402_1005Metric, symbol Device:R
- PPC1: footprint ppc-watch:ppc-board -> powerpic:ppc-board
Connections:
- net VCC: now also R2.2
- net DEBUG renamed CASE
- net CASE: now also D2.2 (A)
- new net: D2.1 (K), R2.1
Other:
- moved on the sheet: C1, C2, C6, PPC1A
